File: filtre-In.sch (KiCad schematic (older format))
At the start: 114 parts, among them P1 BNC Output, P10 BNC, P11 BNC, P12 BNC, P13 BNC, P14 BNC, P16 CONN_01X05, P17 CONN_01X01, P18 CONN_01X01, P19 CONN_01X01, P2 BNC Input, P20 CONN_01X01, P3 CONN_01X08, P4 CONN_01X01, P5 CONN_01X01, P6 CONN_01X01, P7 CONN_01X01, P9 BNC

Commit message: version CAO finale, a priori bonne pour la prod
Parts:
- added C42, C45, C46, C47, C48, C49, C50, C51, C52, C53, C54, C55, C56, C57, C58, C59, C60, C61, C62, C63: C_Small, Capacitors_SMD:C_1825_HandSoldering, symbol C_Small
- R1: footprint Resistors_ThroughHole:R_Axial_DIN0411_L9.9mm_D3.6mm_P12.70mm_Horizontal -> Resistors_THT:R_Axial_DIN0411_L9.9mm_D3.6mm_P12.70mm_Horizontal
Connections:
- net GND: now also C42.1, C45.1, C46.1, C47.1, C48.1, C49.1, C50.1, C51.1, C52.1, C53.1, C54.1, C55.1, C56.1, C57.1, C58.1, C59.1, C60.1, C61.1, C62.1, C63.1
- net at C3.1, L3.1, RL2.1: now also C45.2
- net at C2.1, L3.2, RL1.1: now also C42.2
- net at C6.1, L4.1, RL4.1: now also C47.2
- net at C5.1, L4.2, RL3.1: now also C46.2
- net at C8.1, L5.1, RL6.1: now also C49.2
- net at C7.1, L5.2, RL5.1: now also C48.2
- net at C10.1, L6.1, RL8.1: now also C51.2
- net at C9.1, L6.2, RL7.1: now also C50.2
- net at C12.1, L7.1, RL10.1: now also C53.2
- net at C11.1, L7.2, RL9.1: now also C52.2
- net at C14.1, L8.1, RL12.1: now also C55.2
- net at C13.1, L8.2, RL11.1: now also C54.2
- net at C16.1, L9.1, RL14.1: now also C57.2
- net at C15.1, L9.2, RL13.1: now also C56.2
- net at C18.1, L10.1, RL16.1: now also C59.2
- net at C17.1, L10.2, RL15.1: now also C58.2
- net at C20.1, L11.1, RL18.1: now also C61.2
- net at C19.1, L11.2, RL17.1: now also C60.2
- net at C22.1, L12.1, RL20.1: now also C63.2
- net at C21.1, L12.2, RL19.1: now also C62.2
Other:
- moved on the sheet: C10, C12, C14, C16, C18, C20, C22, C3, C6, C8

Commit message: release from June 12 2017, debugged and checked
Parts:
- P16: footprint Connectors_Molex:Molex_KK-6410-05_05x2.54mm_Straight -> conn_kk100:kk100_22-23-2051
- P3: footprint Connectors_Molex:Molex_KK-6410-08_08x2.54mm_Straight -> conn_kk100:kk100_22-23-2081
Changed lines of the file:
@@
 EESchema Schematic File Version 2
-LIBS:Omron_G5LE
 LIBS:power
 LIBS:conn
 LIBS:device
 LIBS:regul
+LIBS:Omron_G5LE
 LIBS:filtre-In-cache
 EELAYER 25 0
@@
 F 0 "P3" H 4300 6500 50  0000 C CNN
 F 1 "CONN_01X08" V 4400 6050 50  0000 C CNN
-F 2 "Connectors_Molex:Molex_KK-6410-08_08x2.54mm_Straight" H 4300 6050 50  0001 C CNN
+F 2 "conn_kk100:kk100_22-23-2081" H 4300 6050 50  0001 C CNN
 F 3 "" H 4300 6050 50  0000 C CNN
 	1    4300 6050
@@
 F 0 "P16" H 8750 6350 50  0000 C CNN
 F 1 "CONN_01X05" V 8850 6050 50  0000 C CNN
-F 2 "Connectors_Molex:Molex_KK-6410-05_05x2.54mm_Straight" H 8750 6050 50  0001 C CNN
+F 2 "conn_kk100:kk100_22-23-2051" H 8750 6050 50  0001 C CNN
 F 3 "" H 8750 6050 50  0000 C CNN
 	1    8750 6050
